File: hw/ECE445L_Lab7/ECE445L_Lab7.kicad_sch (KiCad schematic)
At the start: 4 parts

Commit message: added reverse engineering for water atomizer
Other:
- company: The University of Texas at Austin -> ECE445L
Changed lines of the file:
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@@
 	(title_block
 		(title "ECE 445L Lab7")
-		(date "2025-01-13")
-		(rev "v1.0.0")
-		(company "The University of Texas at Austin")
+		(date "2026-10-26")
+		(rev "A")
+		(company "ECE445L")
 	)
 	(symbol

Commit message: finished prelim schem
Other:
- sheet Lab7_Input renamed Lab7 IO
- sheet Lab7_Output renamed Lab7 Electromech
- sheet Lab7_microcontroller renamed Lab7 Microcontroller
- sheet Lab7_power renamed Lab7 Power
- sheet Lab7_wifi renamed Lab7 Wifi
Changed lines of the file:
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@@
 	)
 	(sheet
-		(at 38.1 25.4)
-		(size 196.85 20.955)
+		(at 38.735 43.18)
+		(size 31.75 20.955)
 		(exclude_from_sim no)
 		(in_bom yes)
@@
 			(color 255 255 0 1)
 		)
-		(property "Sheetname" "Lab7_power"
-			(at 38.1 24.6884 0)
+		(property "Sheetname" "Lab7 Power"
+			(at 38.735 42.4684 0)
 			(show_name no)
 			(do_not_autoplace no)
@@
 		)
 		(property "Sheetfile" "Lab7_power.kicad_sch"
-			(at 38.1 46.9396 0)
+			(at 38.735 64.7196 0)
 			(show_name no)
 			(do_not_autoplace no)
@@
 	)
 	(sheet
-		(at 169.545 102.87)
+		(at 104.14 103.505)
 		(size 35.56 16.51)
 		(exclude_from_sim no)
@@
 			(color 255 229 191 1)
 		)
-		(property "Sheetname" "Lab7_wifi"
-			(at 169.545 102.1584 0)
+		(property "Sheetname" "Lab7 Wifi"
+			(at 104.14 102.7934 0)
 			(show_name no)
 			(do_not_autoplace no)
@@
 		)
 		(property "Sheetfile" "Lab7_wifi.kicad_sch"
-			(at 169.545 119.9646 0)
+			(at 104.14 120.5996 0)
 			(show_name no)
 			(do_not_autoplace no)
@@
 	)
 	(sheet
-		(at 186.055 63.5)
+		(at 104.775 44.45)
 		(size 40.005 19.685)
 		(exclude_from_sim no)
@@
 			(color 0 255 0 1)
 		)
-		(property "Sheetname" "Lab7_Output"
-			(at 186.055 62.7884 0)
+		(property "Sheetname" "Lab7 Electromech"
+			(at 104.775 43.7384 0)
 			(show_name no)
 			(do_not_autoplace no)
@@
 		)
 		(property "Sheetfile" "Lab7_Output.kicad_sch"
-			(at 186.055 83.7696 0)
+			(at 104.775 64.7196 0)
 			(show_name no)
 			(do_not_autoplace no)
@@
 			(color 0 255 255 1)
 		)
-		(property "Sheetname" "Lab7_microcontroller"
+		(property "Sheetname" "Lab7 Microcontroller"
 			(at 104.775 73.5834 0)
 			(show_name no)
@@
 			(color 0 255 0 1)
 		)
-		(property "Sheetname" "Lab7_Input"
+		(property "Sheetname" "Lab7 IO"
 			(at 39.37 69.7734 0)
 			(show_name no)
