File: hw/ECE445L_Lab7/Lab7_Output.kicad_sch (KiCad schematic)
At the start: 134 parts, among them M1 Motor_DC, M10 Motor_DC, M11 Motor_DC, M12 Motor_DC, M2 Motor_DC, M3 Motor_DC, M4 Motor_DC, M5 Motor_DC, M6 Motor_DC, M7 Motor_DC, M8 Motor_DC, M9 Motor_DC, Q1 NTR4501NT1G, Q10 NTR4501NT1G, Q11 NTR4501NT1G, Q12 NTR4501NT1G, Q13 NTR4501NT1G, Q14 NTR4501NT1G, Q15 NTR4501NT1G, Q2 NTR4501NT1G, Q3 NTR4501NT1G, Q4 NTR4501NT1G, Q5 NTR4501NT1G, Q6 NTR4501NT1G, Q7 NTR4501NT1G, Q8 NTR4501NT1G, Q9 NTR4501NT1G

Commit message: started pcb layout
Parts:
- Motor_In10: renamed from Motor_In11; now not fitted
- Motor_In12, Motor_In2, Motor_In3, Motor_In4, Motor_In5, Motor_In8, Motor_In9, Motor_V_{d}12, Motor_V_{d}2, Motor_V_{d}3, Motor_V_{d}4, Motor_V_{d}5, Motor_V_{d}8, Motor_V_{d}9: now not fitted
- Motor_In7: renamed from Motor_In6; now not fitted
- Motor_V_{d}10: renamed from Motor_V_{d}11; now not fitted
- Motor_V_{d}7: renamed from Motor_V_{d}6; now not fitted
- renumbered Motor_In10 to Motor_In11, Motor_In7 to Motor_In6, Motor_V_{d}10 to Motor_V_{d}11, Motor_V_{d}7 to Motor_V_{d}6, Motor_In15 to Solenoid_In1
Changed lines of the file:
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@@
 		(dnp no)
 		(fields_autoplaced yes)
-		(property "Reference" "Motor_V_{d}7"
-			(at 268.605 58.2929 0)
+		(property "Reference" "Motor_V_{d}6"
+			(at 269.24 58.2929 0)
 			(show_name no)
 			(do_not_autoplace no)
@@
 		)
 		(property "Value" "TestPoint"
-			(at 268.605 60.8329 0)
+			(at 269.24 60.8329 0)
 			(show_name no)
 			(do_not_autoplace no)
@@
 			(project "ECE445L_Lab7"
 				(path "/69b823fd-c065-40ff-9bb9-c5835555f3eb/a500a078-11dc-409b-bff9-a8c35e1dabf8"
-					(reference "Motor_V_{d}7")
+					(reference "Motor_V_{d}6")
 					(unit 1)
 				)
@@
 		(exclude_from_sim no)
 		(in_bom yes)
-		(on_board yes)
+		(on_board no)
 		(in_pos_files yes)
-		(dnp no)
+		(dnp yes)
 		(fields_autoplaced yes)
 		(property "Reference" "Motor_In3"
@@
 		(exclude_from_sim no)
 		(in_bom yes)
-		(on_board yes)
+		(on_board no)
 		(in_pos_files yes)
-		(dnp no)
+		(dnp yes)
 		(fields_autoplaced yes)
 		(property "Reference" "Motor_V_{d}2"
@@
 		(exclude_from_sim no)
 		(in_bom yes)
-		(on_board yes)
+		(on_board no)
 		(in_pos_files yes)
-		(dnp no)
+		(dnp yes)
 		(fields_autoplaced yes)
-		(property "Reference" "Motor_In11"
-			(at 268.605 86.2329 0)
+		(property "Reference" "Motor_In10"
+			(at 269.24 86.2329 0)
 			(show_name no)
 			(do_not_autoplace no)
@@
 		)
 		(property "Value" "TestPoint"
-			(at 268.605 88.7729 0)
+			(at 269.24 88.7729 0)
 			(show_name no)
 			(do_not_autoplace no)
@@
 			(project "ECE445L_Lab7"
 				(path "/69b823fd-c065-40ff-9bb9-c5835555f3eb/a500a078-11dc-409b-bff9-a8c35e1dabf8"
-					(reference "Motor_In11")
+					(reference "Motor_In10")
 					(unit 1)
 				)
@@
 		(exclude_from_sim no)
 		(in_bom yes)
-		(on_board yes)
+		(on_board no)
 		(in_pos_files yes)
-		(dnp no)
+		(dnp yes)
 		(fields_autoplaced yes)
 		(property "Reference" "Motor_V_{d}3"
@@
 		(exclude_from_sim no)
 		(in_bom yes)
-		(on_board yes)
+		(on_board no)
 		(in_pos_files yes)
-		(dnp no)
+		(dnp yes)
 		(fields_autoplaced yes)
-		(property "Reference" "Motor_V_{d}6"
+		(property "Reference" "Motor_V_{d}7"
 			(at 245.11 76.7079 0)
 			(show_name no)
@@
 			(project "ECE445L_Lab7"
 				(path "/69b823fd-c065-40ff-9bb9-c5835555f3eb/a500a078-11dc-409b-bff9-a8c35e1dabf8"
-					(reference "Motor_V_{d}6")
+					(reference "Motor_V_{d}7")
 					(unit 1)
 				)
@@
 		(exclude_from_sim no)
 		(in_bom yes)
-		(on_board yes)
+		(on_board no)
 		(in_pos_files yes)
-		(dnp no)
+		(dnp yes)
 		(fields_autoplaced yes)
 		(property "Reference" "Motor_V_{d}8"
@@
 		(exclude_from_sim no)
 		(in_bom yes)
-		(on_board yes)
+		(on_board no)
 		(in_pos_files yes)
-		(dnp no)
+		(dnp yes)
 		(fields_autoplaced yes)
 		(property "Reference" "Motor_In12"
@@
 		(exclude_from_sim no)
 		(in_bom yes)
-		(on_board yes)
+		(on_board no)
 		(in_pos_files yes)
-		(dnp no)
+		(dnp yes)
 		(fields_autoplaced yes)
 		(property "Reference" "Motor_In5"
@@
 		(exclude_from_sim no)
 		(in_bom yes)
-		(on_board yes)
+		(on_board no)
 		(in_pos_files yes)
-		(dnp no)
+		(dnp yes)
 		(fields_autoplaced yes)
 		(property "Reference" "Motor_In8"
@@
 		(dnp no)
 		(fields_autoplaced yes)
-		(property "Reference" "Motor_V_{d}10"
+		(property "Reference" "Motor_V_{d}11"
 			(at 245.11 112.9029 0)
 			(show_name no)
@@
 			(project "ECE445L_Lab7"
 				(path "/69b823fd-c065-40ff-9bb9-c5835555f3eb/a500a078-11dc-409b-bff9-a8c35e1dabf8"
-					(reference "Motor_V_{d}10")
+					(reference "Motor_V_{d}11")
 					(unit 1)
 				)
@@
 		(exclude_from_sim no)
 		(in_bom yes)
-		(on_board yes)
+		(on_board no)
 		(in_pos_files yes)
-		(dnp no)
+		(dnp yes)
 		(fields_autoplaced yes)
 		(property "Reference" "Motor_V_{d}12"
@@
 		(dnp no)
 		(fields_autoplaced yes)
-		(property "Reference" "Motor_In15"
+		(property "Reference" "Solenoid_In1"
 			(at 270.51 121.7929 0)
 			(show_name no)
@@
 			(project "ECE445L_Lab7"
 				(path "/69b823fd-c065-40ff-9bb9-c5835555f3eb/a500a078-11dc-409b-bff9-a8c35e1dabf8"
-					(reference "Motor_In15")
+					(reference "Solenoid_In1")
 					(unit 1)
 				)
@@
 		(dnp no)
 		(fields_autoplaced yes)
-		(property "Reference" "Motor_In7"
-			(at 268.605 50.0379 0)
+		(property "Reference" "Motor_In6"
+			(at 269.24 50.0379 0)
 			(show_name no)
 			(do_not_autoplace no)
@@
 		)
 		(property "Value" "TestPoint"
-			(at 268.605 52.5779 0)
+			(at 269.24 52.5779 0)
 			(show_name no)
 			(do_not_autoplace no)
@@
 			(project "ECE445L_Lab7"
 				(path "/69b823fd-c065-40ff-9bb9-c5835555f3eb/a500a078-11dc-409b-bff9-a8c35e1dabf8"
-					(reference "Motor_In7")
+					(reference "Motor_In6")
 					(unit 1)
 				)
@@
 		(exclude_from_sim no)
 		(in_bom yes)
-		(on_board yes)
+		(on_board no)
 		(in_pos_files yes)
-		(dnp no)
+		(dnp yes)
 		(fields_autoplaced yes)
 		(property "Reference" "Motor_V_{d}9"
@@
 		(exclude_from_sim no)
 		(in_bom yes)
-		(on_board yes)
+		(on_board no)
 		(in_pos_files yes)
-		(dnp no)
+		(dnp yes)
 		(fields_autoplaced yes)
-		(property "Reference" "Motor_V_{d}11"
-			(at 268.605 94.4879 0)
+		(property "Reference" "Motor_V_{d}10"
+			(at 269.24 94.4879 0)
 			(show_name no)
 			(do_not_autoplace no)
@@
 		)
 		(property "Value" "TestPoint"
-			(at 268.605 97.0279 0)
+			(at 269.24 97.0279 0)
 			(show_name no)
 			(do_not_autoplace no)
@@
 			(project "ECE445L_Lab7"
 				(path "/69b823fd-c065-40ff-9bb9-c5835555f3eb/a500a078-11dc-409b-bff9-a8c35e1dabf8"
-					(reference "Motor_V_{d}11")
+					(reference "Motor_V_{d}10")
 					(unit 1)
 				)
@@
 		(exclude_from_sim no)
 		(in_bom yes)
-		(on_board yes)
+		(on_board no)
 		(in_pos_files yes)
-		(dnp no)
+		(dnp yes)
 		(fields_autoplaced yes)
 		(property "Reference" "Motor_In2"
@@
 		(exclude_from_sim no)
 		(in_bom yes)
-		(on_board yes)
+		(on_board no)
 		(in_pos_files yes)
-		(dnp no)
+		(dnp yes)
 		(fields_autoplaced yes)
-		(property "Reference" "Motor_In6"
+		(property "Reference" "Motor_In7"
 			(at 245.11 68.4529 0)
 			(show_name no)
@@
 			(project "ECE445L_Lab7"
 				(path "/69b823fd-c065-40ff-9bb9-c5835555f3eb/a500a078-11dc-409b-bff9-a8c35e1dabf8"
-					(reference "Motor_In6")
+					(reference "Motor_In7")
 					(unit 1)
 				)
@@
 		(exclude_from_sim no)
 		(in_bom yes)
-		(on_board yes)
+		(on_board no)
 		(in_pos_files yes)
-		(dnp no)
+		(dnp yes)
 		(fields_autoplaced yes)
 		(property "Reference" "Motor_V_{d}5"
@@
 		(exclude_from_sim no)
 		(in_bom yes)
-		(on_board yes)
+		(on_board no)
 		(in_pos_files yes)
-		(dnp no)
+		(dnp yes)
 		(fields_autoplaced yes)
 		(property "Reference" "Motor_V_{d}4"
@@
 		(exclude_from_sim no)
 		(in_bom yes)
-		(on_board yes)
+		(on_board no)
 		(in_pos_files yes)
-		(dnp no)
+		(dnp yes)
 		(fields_autoplaced yes)
 		(property "Reference" "Motor_In9"
@@
 		(exclude_from_sim no)
 		(in_bom yes)
-		(on_board yes)
+		(on_board no)
 		(in_pos_files yes)
-		(dnp no)
+		(dnp yes)
 		(fields_autoplaced yes)
 		(property "Reference" "Motor_In4"
@@
 		(dnp no)
 		(fields_autoplaced yes)
-		(property "Reference" "Motor_In10"
+		(property "Reference" "Motor_In11"
 			(at 245.11 104.6479 0)
 			(show_name no)
@@
 			(project "ECE445L_Lab7"
 				(path "/69b823fd-c065-40ff-9bb9-c5835555f3eb/a500a078-11dc-409b-bff9-a8c35e1dabf8"
-					(reference "Motor_In10")
+					(reference "Motor_In11")
 					(unit 1)
 				)

Commit message: handoff to jonathan until midnight
Parts:
- removed Flywheel_V_{d}2: TestPoint, TestPoint:TestPoint_Keystone_5010-5014_Multipurpose, symbol Connector:TestPoint
- removed SW_{bypass}14: NO, ECE445L:SW_PUSH_6mm, symbol ECE445L:SW_Push
- C_{b}1, C_{b}10, C_{b}11, C_{b}12, C_{b}13, C_{b}14, C_{b}15, C_{b}2, C_{b}3, C_{b}4, C_{b}5, C_{b}6, C_{b}7, C_{b}8, C_{b}9, R_{choke}1, R_{choke}10, R_{choke}11, R_{choke}12, R_{choke}13, R_{choke}14, R_{choke}15, R_{choke}2, R_{choke}3, R_{choke}4, R_{choke}5, R_{choke}6, R_{choke}7, R_{choke}8, R_{choke}9: Distributor Mouser -> Valvano
- D_{flyback}1, D_{flyback}10, D_{flyback}11, D_{flyback}12, D_{flyback}13, D_{flyback}14, D_{flyback}15, D_{flyback}2, D_{flyback}3, D_{flyback}4, D_{flyback}5, D_{flyback}6, D_{flyback}7, D_{flyback}8, D_{flyback}9: value 12V -> ESD5Z12
- Q1, Q10, Q11, Q12, Q13, Q14, Q15, Q2, Q3, Q4, Q5, Q6, Q7, Q8, Q9: Distributor Checkout -> Valvano
- renumbered Flywheel_V_{d}1 to Flywheels_V_{d}1
Connections:
- net V_{d,flywheel 2} is gone; now on net V_{d,flywheels}: D_{flyback}14.2 (A), M_{flywheel,2}1.2 (-), Q14.3 (D)
- net at R_{choke}14.2: now also R_{choke}13.2, SW_{bypass}13.2
- net V_{d,flywheel 1} renamed V_{d,flywheels}
