File: hw/ECE445L_Lab7/Lab7_Output.kicad_sch (KiCad schematic)
At the start: 132 parts, among them M1 Motor_DC, M10 Motor_DC, M11 Motor_DC, M12 Motor_DC, M2 Motor_DC, M3 Motor_DC, M4 Motor_DC, M5 Motor_DC, M6 Motor_DC, M7 Motor_DC, M8 Motor_DC, M9 Motor_DC, Q1 NTR4501NT1G, Q10 NTR4501NT1G, Q11 NTR4501NT1G, Q12 NTR4501NT1G, Q13 NTR4501NT1G, Q14 NTR4501NT1G, Q15 NTR4501NT1G, Q2 NTR4501NT1G, Q3 NTR4501NT1G, Q4 NTR4501NT1G, Q5 NTR4501NT1G, Q6 NTR4501NT1G, Q7 NTR4501NT1G, Q8 NTR4501NT1G, Q9 NTR4501NT1G

Commit message: finished prelim layout for TA review
Parts:
- removed C_{b}13: 4.7u, Capacitor_SMD:C_0603_1608Metric_Pad1.08x0.95mm_HandSolder, symbol ECE445L:C
- removed D_{flyback}13, D_{flyback}14: ESD5Z12, Diode_SMD:D_SOD-523, symbol Device:D_Small
- removed Flywheels_In1, Flywheels_V_{d}1: TestPoint, TestPoint:TestPoint_Keystone_5010-5014_Multipurpose, symbol Connector:TestPoint
- removed M_{flywheel,2}1: Motor_DC, Connector_AMASS:AMASS_XT30U-M_1x02_P5.0mm_Vertical, symbol Motor:Motor_DC
- removed Q13, Q14: NTR4501NT1G, ECE445L:SOT96P237X111-3N, symbol ECE445L:NTR4501NT1G
- removed R_{choke}13, R_{choke}14: 680, Resistor_SMD:R_0603_1608Metric_Pad0.98x0.95mm_HandSolder, symbol Device:R
- removed R_{gate}13, R_{gate}14: 0.25, Resistor_SMD:R_0603_1608Metric_Pad0.98x0.95mm_HandSolder, symbol Device:R
- removed SW_{bypass}13: NO, ECE445L:SW_PUSH_6mm, symbol ECE445L:SW_Push
- added R_{vref}1, R_{vref}2, R_{vref}3, R_{vref}4: 0.5, Resistor_SMD:R_0805_2012Metric_Pad1.20x1.40mm_HandSolder, symbol Device:R
- added U1: DRV8231ADSG, Package_SO:TI_SO-PowerPAD-8, symbol Driver_Motor:DRV8231ADSG
- renumbered M_{flywheel,1}1 to M_{winch}1
Connections:
- net +12V: now also U1.5 (VM); no longer M_{winch}1.1 (+)
- net +3V3: now also U1.4 (VREF)
- net GND: now also R_{vref}1.2, R_{vref}2.2, R_{vref}3.2, R_{vref}4.2, U1.1 (GND), U1.9 (GND)
- net V_{d,flywheels}: no longer names the net of M_{winch}1.2 (-)
- net V_{d,flywheels}: now also U1.8 (OUT2)
- new net: R_{vref}1.1, R_{vref}2.1, R_{vref}3.1, R_{vref}4.1, U1.7 (IPROPI)
- new net: M_{winch}1.1 (+), U1.6 (OUT1)
- new net Winch_{1}: U1.3 (IN1)
- new net Winch_{2}: U1.2 (IN2)
Other:
- moved on the sheet: M_{winch}1, Solenoid_V_{d}1
