File: hw/ECE445L_Lab7/ECE445L_Lab7.kicad_pcb (KiCad board)
At the start: 2 copper layers, 115 x 94 mm, 38 parts, among them J1 JST1.25, J4 Debugger, J5 ZX62D-B-5PA8_30_, J6 Header2, Q1 IRLD024PBF, SW1 UP, SW2 DOWN, SW3 LEFT, SW4 RIGHT, SW5 MODE, SW6 RST, U1 ESP8266-1, U2 Adafruit ST7735R, U4 M0G3507QDGS32RQ1, U5 LP2950-33LPRE3, Y1 16MHz

Commit message: finished prelim schem
Parts:
- removed +3.3V1: +3.3V, ECE445L:Testpoint_1x02_P2.54mm
- removed +5V1: +5V, ECE445L:Testpoint_1x02_P2.54mm
- removed C3, C5: 4.7uF, ECE445L:CP_Radial_Tantal200mil
- removed C4: 10nF, ECE445L:C_Radial_100mil
- removed D1: 1N914, Diode_THT:D_5W_P12.70mm_Horizontal
- removed GND1: GND, ECE445L:Testpoint_1x02_P2.54mm
- removed J1: JST1.25, ECE445L:JST-1x02_1.25mm
- removed J5: ZX62D-B-5PA8_30_, ECE445L:ZX62DB5PA830
- removed J6: Header2, ECE445L:PinHeader_1x02_P2.54mm_Vertical
- removed R3: 47k, ECE445L:R_Axial_DIN0204_L3.6mm_D1.6mm_P7.62mm_Horizontal
- removed R7: 100k, ECE445L:R_Axial_DIN0204_L3.6mm_D1.6mm_P7.62mm_Horizontal
- removed SW1: UP, ECE445L:SW_PUSH_6mm
- removed SW2: DOWN, ECE445L:SW_PUSH_6mm
- removed SW3: LEFT, ECE445L:SW_PUSH_6mm
- removed SW4: RIGHT, ECE445L:SW_PUSH_6mm
- removed SW5: MODE, ECE445L:SW_PUSH_6mm
- removed SW6: RST, ECE445L:SW_PUSH_6mm
- removed U2: Adafruit ST7735R, ECE445L:adafruit_st7735r2
- removed U5: LP2950-33LPRE3, ECE445L:TL431CLPM
- added 12V1: TestPoint, TestPoint:TestPoint_Keystone_5010-5014_Multipurpose, F.Cu at (242.2, 106.7)
- added 3V3: TestPoint, TestPoint:TestPoint_Keystone_5010-5014_Multipurpose, F.Cu at (242.2, 111.8)
- added C_{b,uC}3: 100n, Capacitor_SMD:C_0603_1608Metric_Pad1.08x0.95mm_HandSolder, F.Cu at (236.5, 122.1)
- added C_{b,uC}4: 10u, Capacitor_SMD:C_0603_1608Metric_Pad1.08x0.95mm_HandSolder, F.Cu at (236.5, 124.6)
- added C_{b}1: 4.7u, Capacitor_SMD:C_0603_1608Metric_Pad1.08x0.95mm_HandSolder, F.Cu at (157.7, 145.0)
- added C_{b}10: 4.7u, Capacitor_SMD:C_0603_1608Metric_Pad1.08x0.95mm_HandSolder, F.Cu at (157.7, 167.6)
- added C_{b}11: 4.7u, Capacitor_SMD:C_0603_1608Metric_Pad1.08x0.95mm_HandSolder, F.Cu at (162.0, 145.0)
- added C_{b}12: 4.7u, Capacitor_SMD:C_0603_1608Metric_Pad1.08x0.95mm_HandSolder, F.Cu at (162.0, 147.5)
- added C_{b}13: 4.7u, Capacitor_SMD:C_0603_1608Metric_Pad1.08x0.95mm_HandSolder, F.Cu at (162.0, 150.0)
- added C_{b}14: 4.7u, Capacitor_SMD:C_0603_1608Metric_Pad1.08x0.95mm_HandSolder, F.Cu at (162.0, 152.5)
- added C_{b}15: 4.7u, Capacitor_SMD:C_0603_1608Metric_Pad1.08x0.95mm_HandSolder, F.Cu at (162.0, 155.0)
- added C_{b}2: 4.7u, Capacitor_SMD:C_0603_1608Metric_Pad1.08x0.95mm_HandSolder, F.Cu at (157.7, 147.5)
- added C_{b}3: 4.7u, Capacitor_SMD:C_0603_1608Metric_Pad1.08x0.95mm_HandSolder, F.Cu at (157.7, 150.0)
- added C_{b}4: 4.7u, Capacitor_SMD:C_0603_1608Metric_Pad1.08x0.95mm_HandSolder, F.Cu at (157.7, 152.5)
- added C_{b}5: 4.7u, Capacitor_SMD:C_0603_1608Metric_Pad1.08x0.95mm_HandSolder, F.Cu at (157.7, 155.0)
- added C_{b}6: 4.7u, Capacitor_SMD:C_0603_1608Metric_Pad1.08x0.95mm_HandSolder, F.Cu at (157.7, 157.5)
- added C_{b}7: 4.7u, Capacitor_SMD:C_0603_1608Metric_Pad1.08x0.95mm_HandSolder, F.Cu at (157.7, 160.1)
- added C_{b}8: 4.7u, Capacitor_SMD:C_0603_1608Metric_Pad1.08x0.95mm_HandSolder, F.Cu at (157.7, 162.6)
- added C_{b}9: 4.7u, Capacitor_SMD:C_0603_1608Metric_Pad1.08x0.95mm_HandSolder, F.Cu at (157.7, 165.1)
- added C_{core}2: 0.47u, Capacitor_SMD:C_0603_1608Metric_Pad1.08x0.95mm_HandSolder, F.Cu at (236.5, 127.2)
- added C_{filter}1: 1200u, Capacitor_THT:CP_Radial_D10.0mm_P5.00mm, F.Cu at (245.5, 98.2)
- added C_{pi}1: 4.7u, Capacitor_SMD:C_0603_1608Metric_Pad1.08x0.95mm_HandSolder, F.Cu at (246.9, 112.6)
- added C_{pi}2: 4.7u, Capacitor_SMD:C_0603_1608Metric_Pad1.08x0.95mm_HandSolder, F.Cu at (246.9, 115.1)
- added C_{y}3: 10p, Capacitor_SMD:C_0603_1608Metric_Pad1.08x0.95mm_HandSolder, F.Cu at (236.5, 129.7)
- added C_{y}4: 10p, Capacitor_SMD:C_0603_1608Metric_Pad1.08x0.95mm_HandSolder, F.Cu at (236.5, 132.2)
- added D_{flyback}1: 12V, Diode_SMD:D_SOD-523, F.Cu at (214.2, 157.5)
- added D_{flyback}10: 12V, Diode_SMD:D_SOD-523, F.Cu at (217.8, 164.8)
- added D_{flyback}11: 12V, Diode_SMD:D_SOD-523, F.Cu at (217.8, 167.3)
- added D_{flyback}12: 12V, Diode_SMD:D_SOD-523, F.Cu at (217.8, 169.7)
- added D_{flyback}13: 12V, Diode_SMD:D_SOD-523, F.Cu at (221.4, 157.5)
- added D_{flyback}14: 12V, Diode_SMD:D_SOD-523, F.Cu at (221.4, 159.9)
- added D_{flyback}15: 12V, Diode_SMD:D_SOD-523, F.Cu at (221.4, 162.4)
- added D_{flyback}16: 1N914, Diode_THT:D_5W_P12.70mm_Horizontal, F.Cu at (220.6, 77.8)
- added D_{flyback}17: 1N914, Diode_THT:D_5W_P12.70mm_Horizontal, F.Cu at (220.6, 83.1)
- added D_{flyback}2: 12V, Diode_SMD:D_SOD-523, F.Cu at (214.2, 159.9)
- added D_{flyback}3: 12V, Diode_SMD:D_SOD-523, F.Cu at (214.2, 162.4)
- added D_{flyback}4: 12V, Diode_SMD:D_SOD-523, F.Cu at (214.2, 164.8)
- added D_{flyback}5: 12V, Diode_SMD:D_SOD-523, F.Cu at (214.2, 167.3)
- added D_{flyback}6: 12V, Diode_SMD:D_SOD-523, F.Cu at (214.2, 169.7)
- added D_{flyback}7: 12V, Diode_SMD:D_SOD-523, F.Cu at (217.8, 157.5)
- added D_{flyback}8: 12V, Diode_SMD:D_SOD-523, F.Cu at (217.8, 159.9)
- added D_{flyback}9: 12V, Diode_SMD:D_SOD-523, F.Cu at (217.8, 162.4)
- added F1: Fuse, Fuse:Fuseholder_Cylinder-5x20mm_Wuerth_696103101002-SMD_Horizontal_Open, F.Cu at (131.5, 116.0)
- added Flywheel_V_{d}1: TestPoint, TestPoint:TestPoint_Keystone_5010-5014_Multipurpose, F.Cu at (189.7, 131.2)
- added Flywheel_V_{d}2: TestPoint, TestPoint:TestPoint_Keystone_5010-5014_Multipurpose, F.Cu at (189.7, 136.3)
- added Flywheels_In1: TestPoint, TestPoint:TestPoint_Keystone_5010-5014_Multipurpose, F.Cu at (189.7, 141.3)
- added JP_{Motor}1: Jumper_3_Open, Connector_PinHeader_2.54mm:PinHeader_1x03_P2.54mm_Vertical, F.Cu at (268.5, 132.5)
- added JP_{Motor}2: Jumper_3_Open, Connector_PinHeader_2.54mm:PinHeader_1x03_P2.54mm_Vertical, F.Cu at (197.8, 70.4)
- added JP_{Motor}3: Jumper_3_Open, Connector_PinHeader_2.54mm:PinHeader_1x03_P2.54mm_Vertical, F.Cu at (202.4, 70.4)
- added JP_{Motor}4: Jumper_3_Open, Connector_PinHeader_2.54mm:PinHeader_1x03_P2.54mm_Vertical, F.Cu at (207.0, 70.4)
- added J_{IDReader}1: Conn_01x04, Connector_PinSocket_2.54mm:PinSocket_1x04_P2.54mm_Vertical, F.Cu at (252.1, 70.4)
- added J_{Keypad}1: Conn_01x08, ECE445L:4x4_Matrix_Keypad, F.Cu at (89.8, 139.6)
- added J_{PA14,LED}1: Conn_01x02, Connector_PinSocket_2.54mm:PinSocket_1x02_P2.54mm_Vertical, F.Cu at (220.7, 70.4)
- added J_{PA21,LED}1: Conn_01x02, Connector_PinSocket_2.54mm:PinSocket_1x02_P2.54mm_Vertical, F.Cu at (225.3, 70.4)
- added J_{PA3,LED}1: Conn_01x02, Connector_PinSocket_2.54mm:PinSocket_1x02_P2.54mm_Vertical, F.Cu at (229.9, 70.4)
- added J_{PA7,LED}1: Conn_01x02, Connector_PinSocket_2.54mm:PinSocket_1x02_P2.54mm_Vertical, F.Cu at (234.5, 70.4)
- added J_{USB-C}1: Conn_01x02, Connector_PinHeader_2.54mm:PinHeader_1x02_P2.54mm_Vertical, F.Cu at (247.1, 106.5)
- added J_{atomizer}1: Conn_01x03, Connector_PinSocket_2.54mm:PinSocket_1x03_P2.54mm_Vertical, F.Cu at (211.6, 70.4)
- added J_{flash}2: Debugger, ECE445L:PinHeader_1x04_P2.54mm_Vertical, F.Cu at (241.0, 123.2)
- added J_{test}1: Conn_02x04_Counter_Clockwise, Connector_PinSocket_2.54mm:PinSocket_2x04_P2.54mm_Vertical, F.Cu at (248.1, 123.2)
- added LS2: Speaker, ECE445L:PinHeader_1x02_P2.54mm_Vertical, F.Cu at (197.9, 80.1)
- added L_{filter}1: 10uH, Inductor_SMD:L_Coilcraft_MSS1038-XXX, F.Cu at (235.6, 98.4)
- added M1: Motor_DC, Connector_AMASS:AMASS_XT30U-M_1x02_P5.0mm_Vertical, F.Cu at (190.8, 96.1)
- added M10: Motor_DC, Connector_AMASS:AMASS_XT30U-M_1x02_P5.0mm_Vertical, F.Cu at (203.0, 125.1)
- added M11: Motor_DC, Connector_AMASS:AMASS_XT30U-M_1x02_P5.0mm_Vertical, F.Cu at (215.3, 96.1)
- added M12: Motor_DC, Connector_AMASS:AMASS_XT30U-M_1x02_P5.0mm_Vertical, F.Cu at (215.3, 103.3)
- added M2: Motor_DC, Connector_AMASS:AMASS_XT30U-M_1x02_P5.0mm_Vertical, F.Cu at (190.8, 103.3)
- added M3: Motor_DC, Connector_AMASS:AMASS_XT30U-M_1x02_P5.0mm_Vertical, F.Cu at (190.8, 110.6)
- added M4: Motor_DC, Connector_AMASS:AMASS_XT30U-M_1x02_P5.0mm_Vertical, F.Cu at (190.8, 117.8)
- added M5: Motor_DC, Connector_AMASS:AMASS_XT30U-M_1x02_P5.0mm_Vertical, F.Cu at (190.8, 125.1)
- added M6: Motor_DC, Connector_AMASS:AMASS_XT30U-M_1x02_P5.0mm_Vertical, F.Cu at (203.0, 96.1)
- added M7: Motor_DC, Connector_AMASS:AMASS_XT30U-M_1x02_P5.0mm_Vertical, F.Cu at (203.0, 103.3)
- added M8: Motor_DC, Connector_AMASS:AMASS_XT30U-M_1x02_P5.0mm_Vertical, F.Cu at (203.0, 110.6)
- added M9: Motor_DC, Connector_AMASS:AMASS_XT30U-M_1x02_P5.0mm_Vertical, F.Cu at (203.0, 117.8)
- added M_{feeder}1: Solenoid, Connector_JST:JST_PH_B2B-PH-K_1x02_P2.00mm_Vertical, F.Cu at (180.2, 146.5)
- added M_{flywheel,1}1: Motor_DC, Connector_AMASS:AMASS_XT30U-M_1x02_P5.0mm_Vertical, F.Cu at (215.3, 110.6)
- added M_{flywheel,2}1: Motor_DC, Connector_AMASS:AMASS_XT30U-M_1x02_P5.0mm_Vertical, F.Cu at (215.3, 117.8)
- added Motor_In1: TestPoint, TestPoint:TestPoint_Keystone_5010-5014_Multipurpose, F.Cu at (189.7, 146.4)
- added Motor_In10: TestPoint, TestPoint:TestPoint_Keystone_5010-5014_Multipurpose, F.Cu at (199.8, 131.2)
- added Motor_In11: TestPoint, TestPoint:TestPoint_Keystone_5010-5014_Multipurpose, F.Cu at (199.8, 136.3)
- added Motor_In12: TestPoint, TestPoint:TestPoint_Keystone_5010-5014_Multipurpose, F.Cu at (199.8, 141.3)
- added Motor_In15: TestPoint, TestPoint:TestPoint_Keystone_5010-5014_Multipurpose, F.Cu at (199.8, 146.4)
- added Motor_In2: TestPoint, TestPoint:TestPoint_Keystone_5010-5014_Multipurpose, F.Cu at (189.7, 151.4)
- added Motor_In3: TestPoint, TestPoint:TestPoint_Keystone_5010-5014_Multipurpose, F.Cu at (189.7, 156.5)
- added Motor_In4: TestPoint, TestPoint:TestPoint_Keystone_5010-5014_Multipurpose, F.Cu at (194.7, 131.2)
- added Motor_In5: TestPoint, TestPoint:TestPoint_Keystone_5010-5014_Multipurpose, F.Cu at (194.7, 136.3)
- added Motor_In6: TestPoint, TestPoint:TestPoint_Keystone_5010-5014_Multipurpose, F.Cu at (194.7, 141.3)
- added Motor_In7: TestPoint, TestPoint:TestPoint_Keystone_5010-5014_Multipurpose, F.Cu at (194.7, 146.4)
- added Motor_In8: TestPoint, TestPoint:TestPoint_Keystone_5010-5014_Multipurpose, F.Cu at (194.7, 151.4)
- added Motor_In9: TestPoint, TestPoint:TestPoint_Keystone_5010-5014_Multipurpose, F.Cu at (194.7, 156.5)
- added Motor_V_{d}1: TestPoint, TestPoint:TestPoint_Keystone_5010-5014_Multipurpose, F.Cu at (199.8, 151.4)
- added Motor_V_{d}10: TestPoint, TestPoint:TestPoint_Keystone_5010-5014_Multipurpose, F.Cu at (209.9, 136.3)
- added Motor_V_{d}11: TestPoint, TestPoint:TestPoint_Keystone_5010-5014_Multipurpose, F.Cu at (209.9, 141.3)
- added Motor_V_{d}12: TestPoint, TestPoint:TestPoint_Keystone_5010-5014_Multipurpose, F.Cu at (209.9, 146.4)
- added Motor_V_{d}2: TestPoint, TestPoint:TestPoint_Keystone_5010-5014_Multipurpose, F.Cu at (199.8, 156.5)
- added Motor_V_{d}3: TestPoint, TestPoint:TestPoint_Keystone_5010-5014_Multipurpose, F.Cu at (204.8, 131.2)
- added Motor_V_{d}4: TestPoint, TestPoint:TestPoint_Keystone_5010-5014_Multipurpose, F.Cu at (204.8, 136.3)
- added Motor_V_{d}5: TestPoint, TestPoint:TestPoint_Keystone_5010-5014_Multipurpose, F.Cu at (204.8, 141.3)
- added Motor_V_{d}6: TestPoint, TestPoint:TestPoint_Keystone_5010-5014_Multipurpose, F.Cu at (204.8, 146.4)
- added Motor_V_{d}7: TestPoint, TestPoint:TestPoint_Keystone_5010-5014_Multipurpose, F.Cu at (204.8, 151.4)
- added Motor_V_{d}8: TestPoint, TestPoint:TestPoint_Keystone_5010-5014_Multipurpose, F.Cu at (204.8, 156.5)
- added Motor_V_{d}9: TestPoint, TestPoint:TestPoint_Keystone_5010-5014_Multipurpose, F.Cu at (209.9, 131.2)
- added Q10: NTR4501NT1G, ECE445L:SOT96P237X111-3N, F.Cu at (219.8, 144.8)
- added Q11: NTR4501NT1G, ECE445L:SOT96P237X111-3N, F.Cu at (219.8, 149.3)
- added Q12: NTR4501NT1G, ECE445L:SOT96P237X111-3N, F.Cu at (219.8, 153.9)
- added Q13: NTR4501NT1G, ECE445L:SOT96P237X111-3N, F.Cu at (224.8, 131.0)
- added Q14: NTR4501NT1G, ECE445L:SOT96P237X111-3N, F.Cu at (224.8, 135.6)
- added Q15: NTR4501NT1G, ECE445L:SOT96P237X111-3N, F.Cu at (224.8, 140.2)
- added Q16: NTR4501NT1G, ECE445L:SOT96P237X111-3N, F.Cu at (202.7, 80.0)
- added Q17: NTR4501NT1G, ECE445L:SOT96P237X111-3N, F.Cu at (202.7, 84.6)
- added Q2: NTR4501NT1G, ECE445L:SOT96P237X111-3N, F.Cu at (214.9, 135.6)
- added Q3: NTR4501NT1G, ECE445L:SOT96P237X111-3N, F.Cu at (214.9, 140.2)
- added Q4: NTR4501NT1G, ECE445L:SOT96P237X111-3N, F.Cu at (214.9, 144.8)
- added Q5: NTR4501NT1G, ECE445L:SOT96P237X111-3N, F.Cu at (214.9, 149.3)
- added Q6: NTR4501NT1G, ECE445L:SOT96P237X111-3N, F.Cu at (214.9, 153.9)
- added Q7: NTR4501NT1G, ECE445L:SOT96P237X111-3N, F.Cu at (219.8, 131.0)
- added Q8: NTR4501NT1G, ECE445L:SOT96P237X111-3N, F.Cu at (219.8, 135.6)
- added Q9: NTR4501NT1G, ECE445L:SOT96P237X111-3N, F.Cu at (219.8, 140.2)
- added R_{PU}2: 10k, Resistor_SMD:R_0805_2012Metric_Pad1.20x1.40mm_HandSolder, F.Cu at (202.6, 88.4)
- added R_{choke}1: 680, Resistor_SMD:R_0603_1608Metric_Pad0.98x0.95mm_HandSolder, F.Cu at (265.9, 128.0)
- added R_{choke}10: 680, Resistor_SMD:R_0603_1608Metric_Pad0.98x0.95mm_HandSolder, F.Cu at (166.4, 155.0)
- added R_{choke}11: 680, Resistor_SMD:R_0603_1608Metric_Pad0.98x0.95mm_HandSolder, F.Cu at (166.4, 157.5)
- added R_{choke}12: 680, Resistor_SMD:R_0603_1608Metric_Pad0.98x0.95mm_HandSolder, F.Cu at (166.4, 160.1)
- added R_{choke}13: 680, Resistor_SMD:R_0603_1608Metric_Pad0.98x0.95mm_HandSolder, F.Cu at (166.4, 162.6)
- added R_{choke}14: 680, Resistor_SMD:R_0603_1608Metric_Pad0.98x0.95mm_HandSolder, F.Cu at (166.4, 165.1)
- added R_{choke}15: 680, Resistor_SMD:R_0603_1608Metric_Pad0.98x0.95mm_HandSolder, F.Cu at (166.4, 167.6)
- added R_{choke}2: 680, Resistor_SMD:R_0603_1608Metric_Pad0.98x0.95mm_HandSolder, F.Cu at (162.0, 160.1)
- added R_{choke}3: 680, Resistor_SMD:R_0603_1608Metric_Pad0.98x0.95mm_HandSolder, F.Cu at (162.0, 162.6)
- added R_{choke}4: 680, Resistor_SMD:R_0603_1608Metric_Pad0.98x0.95mm_HandSolder, F.Cu at (162.0, 165.1)
- added R_{choke}5: 680, Resistor_SMD:R_0603_1608Metric_Pad0.98x0.95mm_HandSolder, F.Cu at (162.0, 167.6)
- added R_{choke}6: 680, Resistor_SMD:R_0603_1608Metric_Pad0.98x0.95mm_HandSolder, F.Cu at (166.4, 145.0)
- added R_{choke}7: 680, Resistor_SMD:R_0603_1608Metric_Pad0.98x0.95mm_HandSolder, F.Cu at (166.4, 147.5)
- added R_{choke}8: 680, Resistor_SMD:R_0603_1608Metric_Pad0.98x0.95mm_HandSolder, F.Cu at (166.4, 150.0)
- added R_{choke}9: 680, Resistor_SMD:R_0603_1608Metric_Pad0.98x0.95mm_HandSolder, F.Cu at (166.4, 152.5)
- added R_{filter}1: 0.25, Resistor_SMD:R_0603_1608Metric_Pad0.98x0.95mm_HandSolder, F.Cu at (246.9, 117.6)
- added R_{gate}1: 0.25, Resistor_SMD:R_0603_1608Metric_Pad0.98x0.95mm_HandSolder, F.Cu at (268.5, 129.0)
- added R_{gate}10: 0.25, Resistor_SMD:R_0603_1608Metric_Pad0.98x0.95mm_HandSolder, F.Cu at (170.7, 167.6)
- added R_{gate}11: 0.25, Resistor_SMD:R_0603_1608Metric_Pad0.98x0.95mm_HandSolder, F.Cu at (175.1, 145.0)
- added R_{gate}12: 0.25, Resistor_SMD:R_0603_1608Metric_Pad0.98x0.95mm_HandSolder, F.Cu at (175.1, 147.5)
- added R_{gate}13: 0.25, Resistor_SMD:R_0603_1608Metric_Pad0.98x0.95mm_HandSolder, F.Cu at (175.1, 150.0)
- added R_{gate}14: 0.25, Resistor_SMD:R_0603_1608Metric_Pad0.98x0.95mm_HandSolder, F.Cu at (175.1, 152.5)
- added R_{gate}15: 0.25, Resistor_SMD:R_0603_1608Metric_Pad0.98x0.95mm_HandSolder, F.Cu at (175.1, 155.0)
- added R_{gate}2: 0.25, Resistor_SMD:R_0603_1608Metric_Pad0.98x0.95mm_HandSolder, F.Cu at (170.7, 147.5)
- added R_{gate}3: 0.25, Resistor_SMD:R_0603_1608Metric_Pad0.98x0.95mm_HandSolder, F.Cu at (170.7, 150.0)
- added R_{gate}4: 0.25, Resistor_SMD:R_0603_1608Metric_Pad0.98x0.95mm_HandSolder, F.Cu at (170.7, 152.5)
- added R_{gate}5: 0.25, Resistor_SMD:R_0603_1608Metric_Pad0.98x0.95mm_HandSolder, F.Cu at (170.7, 155.0)
- added R_{gate}6: 0.25, Resistor_SMD:R_0603_1608Metric_Pad0.98x0.95mm_HandSolder, F.Cu at (170.7, 157.5)
- added R_{gate}7: 0.25, Resistor_SMD:R_0603_1608Metric_Pad0.98x0.95mm_HandSolder, F.Cu at (170.7, 160.1)
- added R_{gate}8: 0.25, Resistor_SMD:R_0603_1608Metric_Pad0.98x0.95mm_HandSolder, F.Cu at (170.7, 162.6)
- added R_{gate}9: 0.25, Resistor_SMD:R_0603_1608Metric_Pad0.98x0.95mm_HandSolder, F.Cu at (170.7, 165.1)
- added RxD_{ID}1: TestPoint, TestPoint:TestPoint_Keystone_5010-5014_Multipurpose, F.Cu at (252.4, 82.8)
- added SPI_{CS}1: TestPoint, TestPoint:TestPoint_Keystone_5010-5014_Multipurpose, F.Cu at (231.8, 123.4)
- added SPI_{SCK}1: TestPoint, TestPoint:TestPoint_Keystone_5010-5014_Multipurpose, F.Cu at (231.8, 128.5)
- added SW_{bypass}1: NO, ECE445L:SW_PUSH_6mm, F.Cu at (157.5, 94.5)
- added SW_{bypass}10: NO, ECE445L:SW_PUSH_6mm, F.Cu at (168.1, 120.1)
- added SW_{bypass}11: NO, ECE445L:SW_PUSH_6mm, F.Cu at (168.1, 128.7)
- added SW_{bypass}12: NO, ECE445L:SW_PUSH_6mm, F.Cu at (168.1, 137.2)
- added SW_{bypass}13: NO, ECE445L:SW_PUSH_6mm, F.Cu at (178.6, 94.5)
- added SW_{bypass}14: NO, ECE445L:SW_PUSH_6mm, F.Cu at (178.6, 103.0)
- added SW_{bypass}15: NO, ECE445L:SW_PUSH_6mm, F.Cu at (178.6, 111.6)
- added SW_{bypass}2: NO, ECE445L:SW_PUSH_6mm, F.Cu at (157.5, 103.0)
- added SW_{bypass}3: NO, ECE445L:SW_PUSH_6mm, F.Cu at (157.5, 111.6)
- added SW_{bypass}4: NO, ECE445L:SW_PUSH_6mm, F.Cu at (157.5, 120.1)
- added SW_{bypass}5: NO, ECE445L:SW_PUSH_6mm, F.Cu at (157.5, 128.7)
- added SW_{bypass}6: NO, ECE445L:SW_PUSH_6mm, F.Cu at (157.5, 137.2)
- added SW_{bypass}7: NO, ECE445L:SW_PUSH_6mm, F.Cu at (168.1, 94.5)
- added SW_{bypass}8: NO, ECE445L:SW_PUSH_6mm, F.Cu at (168.1, 103.0)
- added SW_{bypass}9: NO, ECE445L:SW_PUSH_6mm, F.Cu at (168.1, 111.6)
- added Solenoid_V_{d}1: TestPoint, TestPoint:TestPoint_Keystone_5010-5014_Multipurpose, F.Cu at (209.9, 151.4)
- added TFT1: Adafruit ST7735R, ECE445L:adafruit_st7735r2, F.Cu at (88.0, 42.7)
- added TFT2: HiLetGo_ST7735R, ECE445L:hiletgo_st7735r2, F.Cu at (89.8, 170.2)
- added TxD_{ID}1: TestPoint, TestPoint:TestPoint_Keystone_5010-5014_Multipurpose, F.Cu at (252.4, 87.9)
- added U_{3V3DC}1: RBT05W24S12, Converter_DCDC:Converter_DCDC_TRACO_TSR0.5-24xx_TSR0.5-24xxx_THT, F.Cu at (233.0, 108.7)
- added U_{Decoder}1: MC14514BDWR2G, ECE445L:SOIC-24WB_ONS, F.Cu at (243.3, 76.6)
- added Y2: 16MHz, ECE445L:ABM3, F.Cu at (246.9, 136.6)
- added uC2: M0G3507QDGS32RQ1, ECE445L:VSSOP_0.5mm_32pin_handsolder, F.Cu at (273.8, 138.4)
- added uC_{1}←uC_{2}1: TestPoint, TestPoint:TestPoint_Keystone_5010-5014_Multipurpose, F.Cu at (231.8, 133.5)
- added uC_{1}→uC_{2}1: TestPoint, TestPoint:TestPoint_Keystone_5010-5014_Multipurpose, F.Cu at (231.8, 138.6)
- C_{b,uC}1: renamed from C8; value 0.1uF -> 100n; footprint ECE445L:C_Radial_100mil -> Capacitor_SMD:C_0603_1608Metric_Pad1.08x0.95mm_HandSolder
- C_{b,uC}2: renamed from C7; value 10uF -> 10u; footprint ECE445L:C_Radial_100mil -> Capacitor_SMD:C_0603_1608Metric_Pad1.08x0.95mm_HandSolder
- C_{b}16: renamed from C1; value 100nF -> 100n; footprint ECE445L:C_Radial_100mil -> Capacitor_SMD:C_0603_1608Metric_Pad1.08x0.95mm_HandSolder
- C_{b}17: renamed from C2; value 4.7uF -> 4.7u; footprint ECE445L:CP_Radial_Tantal200mil -> Capacitor_SMD:C_0603_1608Metric_Pad1.08x0.95mm_HandSolder
- C_{core}1: renamed from C9; value 0.47uF -> 0.47u; footprint ECE445L:C_Radial_100mil -> Capacitor_SMD:C_0603_1608Metric_Pad1.08x0.95mm_HandSolder
- C_{y}1: renamed from C10; value 10pF -> 10p; footprint ECE445L:C_Radial_100mil -> Capacitor_SMD:C_0603_1608Metric_Pad1.08x0.95mm_HandSolder
- C_{y}2: renamed from C11; value 10pF -> 10p; footprint ECE445L:C_Radial_100mil -> Capacitor_SMD:C_0603_1608Metric_Pad1.08x0.95mm_HandSolder
- Q1: value IRLD024PBF -> NTR4501NT1G; footprint ECE445L:DIP920W60P254L490H457Q4N -> ECE445L:SOT96P237X111-3N
- R_{PU}1: renamed from R1; footprint ECE445L:R_Axial_DIN0204_L3.6mm_D1.6mm_P7.62mm_Horizontal -> Resistor_SMD:R_0805_2012Metric_Pad1.20x1.40mm_HandSolder
- moved Q1 201.2 mm to (269.5, 125.2), turned to 90 degrees
- moved uC1 180.1 mm to (262.1, 138.5)
- moved LS1 116.4 mm to (193.2, 80.1)
- moved Y1 90.6 mm to (201.2, 17.4)
- moved C_{b}17 90.6 mm to (207.8, 58.9)
- moved J_{flash}1 90.6 mm to (201.5, 26.4)
- moved R_{PU}1 90.6 mm to (197.0, 56.3)
- moved C_{b}16 90.6 mm to (216.2, 57.1)
- moved C_{b,uC}1 86.0 mm to (184.6, 37.4)
- moved C_{b,uC}2 86.0 mm to (184.6, 32.8)
- moved C_{core}1 86.0 mm to (184.6, 41.9)
- moved C_{y}1 86.0 mm to (184.6, 46.5)
- moved C_{y}2 86.0 mm to (184.6, 51.0)
- moved ESP8266 41.8 mm to (165.0, 46.9)
- moved H1 41.0 mm to (66.2, 60.8)
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- renumbered U1 to ESP8266, J4 to J_{flash}1, U4 to uC1
Connections:
- net Net-(U4-VCORE) renamed /Lab7 Microcontroller/uC_{1} - V_{core}
- net PA5/HFXIN renamed uC_{1} - HFXIN
- net PA6/HFXOUT renamed uC_{1} - HFXOUT
- net SWCLK renamed /Lab7 Microcontroller/uC_{1} - SWCLK
- net SWDIO renamed /Lab7 Microcontroller/uC_{1} - SWDIO
- C_{b}16 pad 1: unconnected-(C1-Pad1) -> +3V3
- C_{b}16 pad 2: unconnected-(C1-Pad2) -> GND
- C_{b}17 pad 1: unconnected-(C2-Pad1) -> +3V3
- C_{b}17 pad 2: unconnected-(C2-Pad2) -> GND
- ESP8266 pad 1: unconnected-(U1-RxD-Pad1) -> uC_{1} - ESP RxD
- ESP8266 pad 2: unconnected-(U1-GPIO0-Pad2) -> +3V3
- ESP8266 pad 3: unconnected-(U1-GPIO2-Pad3) -> uC_{1} - ESP Light
- ESP8266 pad 4: unconnected-(U1-GND-Pad4) -> GND
- ESP8266 pad 5: unconnected-(U1-TxD-Pad5) -> uC_{1} - ESP TxD
- ESP8266 pad 6: unconnected-(U1-Ch_PD-Pad6) -> Net-(ESP8266-Ch_PD)
- ESP8266 pad 7: unconnected-(U1-Reset-Pad7) -> uC_{1} - ESP RST
- ESP8266 pad 8: unconnected-(U1-Vcc-Pad8) -> +3V3
- Q1 pad 1: unconnected-(Q1-D-Pad1) -> Net-(Q1-G)
- Q1 pad 2: unconnected-(Q1-D-Pad2) -> GND
- Q1 pad 3: unconnected-(Q1-G-Pad3) -> /Lab7 Electromech/V_{d,motor 1}
- R_{PU}1 pad 1: unconnected-(R1-Pad1) -> +3V3
- R_{PU}1 pad 2: unconnected-(R1-Pad2) -> Net-(ESP8266-Ch_PD)
- uC1 pad 1: PA26 -> Keypad - R4
- uC1 pad 10: PA3 -> Keypad - C3
- uC1 pad 11: PA4 -> Keypad - R1
- uC1 pad 14: PA7 -> Keypad - R2
- uC1 pad 15: PA8/SPI0_CS0 -> ID Scan - TxD
- uC1 pad 16: PA9 -> ID Scan - RxD
- uC1 pad 17: PA10 -> /Lab7 Microcontroller/uC SPI - uC_{1} ← uC_{2}
- uC1 pad 18: PA11/SPI0_SCK -> Keypad - C4
- uC1 pad 19: PA12 -> uC SPI - SCK
- uC1 pad 2: PA27/SPI1_CS1 -> Adafruit - CS
- uC1 pad 20: PA13/TFT_D/C -> Adafruit - D/C
- uC1 pad 21: PA14/SPI0_PICO -> /Lab7 Microcontroller/uC SPI - uC_{1} → uC_{2}
- uC1 pad 22: PA15/DACOUT -> uC_{1} - Speaker
- uC1 pad 23: PA16/SPI1_POCI -> uC_{1} - ESP Light
- uC1 pad 24: PA17/SPI1_CLK -> Adafruit - SCK
- uC1 pad 25: PA18/SPI1_PICO -> Adafruit - MOSI
- uC1 pad 28: PA21 -> uC_{1} - ESP TxD
- uC1 pad 29: PA22 -> uC_{1} - ESP RxD
- uC1 pad 30: PA23 -> Keypad - R3
- uC1 pad 31: PA24/TFT_RESET -> Adafruit - RST
- uC1 pad 32: PA25/SPI1_CS3 -> uC_{1} - ESP RST
- uC1 pad 4: PA0 -> Keypad - C1
- uC1 pad 5: PA1 -> Keypad - C2
- uC1 pad 6: Net-(U4-NRST) -> unconnected-(uC1-NRST-Pad6)
- uC1 pad 9: PA2 -> uC SPI - CS
Other:
- board size 115 x 94 mm -> 88.5 x 94 mm
- copper layers 2 -> 4

Commit message: started pcb layout
Parts:
- removed Motor_In10, Motor_In12, Motor_In15, Motor_In2, Motor_In3, Motor_In4, Motor_In5, Motor_In7, Motor_In8, Motor_In9, Motor_V_{d}10, Motor_V_{d}12, Motor_V_{d}2, Motor_V_{d}3, Motor_V_{d}4, Motor_V_{d}5, Motor_V_{d}7, Motor_V_{d}8, Motor_V_{d}9: TestPoint, TestPoint:TestPoint_Keystone_5010-5014_Multipurpose
- added J_{atomizer}2: Conn_01x03, Connector_PinSocket_2.54mm:PinSocket_1x03_P2.54mm_Vertical, F.Cu at (255.3, 45.5)
- added Q18: NTR4501NT1G, ECE445L:SOT96P237X111-3N, F.Cu at (239.2, 148.1)
- added Q19: NTR4501NT1G, ECE445L:SOT96P237X111-3N, F.Cu at (239.2, 152.7)
- added Q20: NTR4501NT1G, ECE445L:SOT96P237X111-3N, F.Cu at (239.2, 157.3)
- added Q21: NTR4501NT1G, ECE445L:SOT96P237X111-3N, F.Cu at (239.2, 161.9)
- added R_{I_lim}1: R, Resistor_SMD:R_0603_1608Metric_Pad0.98x0.95mm_HandSolder, F.Cu at (250.8, 44.4)
- added R_{I_lim}2: R, Resistor_SMD:R_0603_1608Metric_Pad0.98x0.95mm_HandSolder, F.Cu at (250.8, 47.0)
- added R_{I_lim}3: R, Resistor_SMD:R_0603_1608Metric_Pad0.98x0.95mm_HandSolder, F.Cu at (250.8, 49.5)
- added R_{I_lim}4: R, Resistor_SMD:R_0603_1608Metric_Pad0.98x0.95mm_HandSolder, F.Cu at (250.8, 52.0)
- added Solenoid_In1: TestPoint, TestPoint:TestPoint_Keystone_5010-5014_Multipurpose, F.Cu at (189.5, 158.2)
- D_{flyback}16, D_{flyback}17: footprint Diode_THT:D_5W_P12.70mm_Horizontal -> Diode_SMD:D_SOD-882D
- ESP8266, M1, M10, M11, M12, M2, M3, M4, M5, M6, M7, M8, M9, M_{flywheel,1}1, M_{flywheel,2}1, SW_{bypass}1, SW_{bypass}2: moved to B.Cu
- F1: footprint Fuse:Fuseholder_Cylinder-5x20mm_Wuerth_696103101002-SMD_Horizontal_Open -> ECE445L:WR-FSH_THT_2; moved to B.Cu
- moved M_{flywheel,2}1 142.8 mm to (75.1, 90.3), turned to 90 degrees
- moved M10 137.0 mm to (67.9, 102.5), turned to 90 degrees
- moved M_{flywheel,1}1 134.4 mm to (82.4, 90.3), turned to 90 degrees
- moved M9 128.8 mm to (75.1, 102.5), turned to 90 degrees
- moved M12 126.3 mm to (89.6, 90.3), turned to 90 degrees
- moved M5 123.3 mm to (67.9, 114.8), turned to 90 degrees
- moved SW_{bypass}2 122.2 mm to (276.7, 130.2)
- moved M8 120.9 mm to (82.4, 102.5), turned to 90 degrees
- moved R_{choke}2 119.2 mm to (276.9, 128.2), turned to 180 degrees
- moved M11 118.5 mm to (96.9, 90.3), turned to 90 degrees
- moved M4 115.7 mm to (75.1, 114.8), turned to 90 degrees
- moved M7 113.4 mm to (89.6, 102.5), turned to 90 degrees
- moved SW_{bypass}1 113.3 mm to (266.0, 127.3)
- moved R_{gate}2 110.2 mm to (279.5, 129.4), turned to -90 degrees
- moved M3 108.5 mm to (82.4, 114.8), turned to 90 degrees
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Connections:
- J_{PA14,LED}1 pad 1: PA14/LG3 -> Net-(J_{PA14,LED}1-Pin_1)
- J_{PA14,LED}1 pad 2: GND -> Net-(J_{PA14,LED}1-Pin_2)
- J_{PA21,LED}1 pad 1: PA21/LG4 -> Net-(J_{PA21,LED}1-Pin_1)
- J_{PA21,LED}1 pad 2: GND -> Net-(J_{PA21,LED}1-Pin_2)
- J_{PA3,LED}1 pad 1: PA3/LG1 -> Net-(J_{PA3,LED}1-Pin_1)
- J_{PA3,LED}1 pad 2: GND -> Net-(J_{PA3,LED}1-Pin_2)
- J_{PA7,LED}1 pad 1: PA7/LG2 -> Net-(J_{PA7,LED}1-Pin_1)
- J_{PA7,LED}1 pad 2: GND -> Net-(J_{PA7,LED}1-Pin_2)
- Motor_In11 pad 1: Motor_{10} -> Motor_{11}
- Motor_In6 pad 1: Motor_{7} -> Motor_{6}
- Motor_V_{d}11 pad 1: /Lab7 Electromech/V_{d,motor 10} -> /Lab7 Electromech/V_{d,motor 11}
- Motor_V_{d}6 pad 1: /Lab7 Electromech/V_{d,motor 7} -> /Lab7 Electromech/V_{d,motor 6}

Commit message: gave up on test branch
Parts:
- SW_{bypass}3, SW_{bypass}4, U_{Decoder}1: moved to B.Cu
- moved M10 238.2 mm to (296.5, 35.7)
- moved M11 238.2 mm to (325.5, 23.5)
- moved M12 238.2 mm to (318.2, 23.5)
- moved M5 238.2 mm to (296.5, 48.0)
- moved M6 238.2 mm to (325.5, 35.7)
- moved M7 238.2 mm to (318.2, 35.7)
- moved M8 238.2 mm to (311.0, 35.7)
- moved M9 238.2 mm to (303.7, 35.7)
- moved M_{flywheel,1}1 238.2 mm to (311.0, 23.5)
- moved M_{flywheel,2}1 238.2 mm to (303.7, 23.5)
- moved Q1 181.8 mm to (91.2, 85.9), turned to 180 degrees
- moved SW_{bypass}2 180.6 mm to (102.7, 81.6), turned to -90 degrees
- moved R_{gate}1 180.0 mm to (92.2, 88.6), turned to 0 degrees
- moved JP_{Motor}1 180.0 mm to (92.4, 91.3)
- moved JP_{Motor}3 178.2 mm to (93.2, 117.1)
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Other:
- board size 88.5 x 94 mm -> 101.6 x 94 mm
- board text added: "Decode - Direct"
- board text added: "Direct - Decode"

Commit message: handoff to jonathan until midnight
Parts:
- removed Flywheel_V_{d}1, Flywheel_V_{d}2: TestPoint, TestPoint:TestPoint_Keystone_5010-5014_Multipurpose
- removed SW_{bypass}14: NO, ECE445L:SW_PUSH_6mm
- added Flywheels_V_{d}1: TestPoint, TestPoint:TestPoint_Keystone_5010-5014_Multipurpose, F.Cu at (143.5, 114.5)
- C_{b,uC}1, C_{b,uC}2, C_{b,uC}3, C_{b,uC}4, C_{b}17, C_{core}1, C_{core}2, C_{filter}1, J_{PA14,LED}1, J_{PA21,LED}1, J_{PA3,LED}1, J_{PA7,LED}1, J_{USB-C}1, J_{flash}1, J_{flash}2, LS1, LS2, M_{feeder}1, R_{filter}1, SW_{bypass}10, SW_{bypass}11, SW_{bypass}12, SW_{bypass}13, SW_{bypass}15, SW_{bypass}5, SW_{bypass}6, SW_{bypass}7, SW_{bypass}8, SW_{bypass}9: moved to B.Cu
- D_{flyback}1, D_{flyback}10, D_{flyback}11, D_{flyback}12, D_{flyback}13, D_{flyback}14, D_{flyback}15, D_{flyback}2, D_{flyback}3, D_{flyback}4, D_{flyback}5, D_{flyback}6, D_{flyback}7, D_{flyback}8, D_{flyback}9: value 12V -> ESD5Z12
- D_{flyback}16, D_{flyback}17: value 1N914 -> PE1403M1Q
- U_{3V3DC}1: footprint Converter_DCDC:Converter_DCDC_TRACO_TSR0.5-24xx_TSR0.5-24xxx_THT -> ECE445L:N78032C; moved to B.Cu
- moved M6 303.8 mm to (35.2, 125.4), turned to 0 degrees
- moved M7 298.8 mm to (35.2, 131.6), turned to 0 degrees
- moved M10 288.7 mm to (35.3, 158.8), turned to 0 degrees
- moved M5 266.0 mm to (35.2, 97.8), turned to 0 degrees
- moved M11 243.0 mm to (123.3, 158.3), turned to 180 degrees
- moved M_{flywheel,1}1 234.9 mm to (123.3, 164.8), turned to 180 degrees
- moved M_{flywheel,2}1 233.0 mm to (123.3, 171.0), turned to 180 degrees
- moved M8 210.6 mm to (123.2, 131.1), turned to 180 degrees
- moved M12 208.5 mm to (123.2, 97.3), turned to 180 degrees
- moved M9 201.3 mm to (123.3, 124.9), turned to 180 degrees
- moved C_{pi}2 194.8 mm to (61.8, 175.7), turned to 90 degrees
- moved C_{pi}1 194.7 mm to (61.6, 172.3), turned to -90 degrees
- moved D_{flyback}16 194.5 mm to (52.9, 176.3), turned to 180 degrees
- moved Q15 189.4 mm to (37.1, 165.2), turned to 180 degrees
- moved D_{flyback}5 188.4 mm to (38.1, 100.2)
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Connections:
- D_{flyback}13 pad 2: /Lab7 Electromech/V_{d,flywheel 1} -> /Lab7 Electromech/V_{d,flywheels}
- D_{flyback}14 pad 2: /Lab7 Electromech/V_{d,flywheel 2} -> /Lab7 Electromech/V_{d,flywheels}
- M_{flywheel,1}1 pad 2: /Lab7 Electromech/V_{d,flywheel 1} -> /Lab7 Electromech/V_{d,flywheels}
- M_{flywheel,2}1 pad 2: /Lab7 Electromech/V_{d,flywheel 2} -> /Lab7 Electromech/V_{d,flywheels}
- Q13 pad 3: /Lab7 Electromech/V_{d,flywheel 1} -> /Lab7 Electromech/V_{d,flywheels}
- Q14 pad 3: /Lab7 Electromech/V_{d,flywheel 2} -> /Lab7 Electromech/V_{d,flywheels}
- R_{choke}14 pad 2: Net-(R_{choke}14-Pad2) -> Net-(R_{choke}13-Pad2)
Other:
- board size 101.6 x 94 mm -> 147.1 x 184.3 mm
- copper layers 4 -> 2

Commit message: Worked on PCB layou/route while Egan was busy
Parts:
- R_{filter}1: moved to F.Cu
- moved J_{PA7,LED}1 250.9 mm to (42.3, 36.4)
- moved Q19 250.9 mm to (37.7, 37.9)
- moved R_{I_lim}2 250.9 mm to (41.5, 38.3)
- moved Q18 250.0 mm to (37.6, 27.9)
- moved J_{PA3,LED}1 250.0 mm to (42.1, 26.4)
- moved R_{I_lim}1 250.0 mm to (41.4, 28.1)
- moved J_{PA21,LED}1 240.9 mm to (41.8, 57.1)
- moved Q21 240.9 mm to (37.6, 58.5)
- moved R_{I_lim}4 240.9 mm to (41.4, 58.6)
- moved J_{PA14,LED}1 229.3 mm to (42.0, 46.5)
- moved Q20 229.3 mm to (37.6, 48.1)
- moved R_{I_lim}3 229.3 mm to (41.4, 48.5)
- moved 3V3 218.8 mm to (38.1, 190.5)
- moved 12V1 211.3 mm to (48.3, 190.5)
- moved H2 183.1 mm to (24.0, 192.2)
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Routing:
- net +3V3: track 0.00 -> 225.6 mm, vias 0 -> 9
- net GND: track 0.00 -> 116.6 mm, vias 0 -> 9
- net Motor_{1}: track 0.00 -> 111.7 mm
- net PA3/LG1: track 0.00 -> 107.9 mm, vias 0 -> 1
- net PA7/LG2: track 0.00 -> 104.3 mm, vias 0 -> 1
- net PA14/LG3: track 0.00 -> 97.3 mm, vias 0 -> 1
- net Motor_{2}: track 0.00 -> 89.1 mm
- net PA21/LG4: track 0.00 -> 88.8 mm
- net /Lab7 IO/D_{Motor}2: track 0.00 -> 87.7 mm, vias 0 -> 2
- net uC_{1} - Speaker: track 0.00 -> 85.9 mm, vias 0 -> 2
- net /Lab7 IO/D_{Motor}1: track 0.00 -> 82.0 mm
- net uC_{2} - Motor_{2}: track 0.00 -> 35.2 mm, vias 0 -> 2
- net uC_{2} - Motor_{1}: track 0.00 -> 30.9 mm
- net /Lab7 Electromech/V_{d,motor 6}: track 0.00 -> 29.9 mm
- net /Lab7 Electromech/V_{d,motor 1}: track 0.00 -> 28.7 mm
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- added copper zone on B.Cu, net +12V
- added copper zone on F.Cu, net +12V
- added copper zone on F.Cu, net +3V3
- added copper zone on B.Cu, net GND

Commit message: finished prelim layout for TA review
Parts:
- removed C_{b}13: 4.7u, Capacitor_SMD:C_0603_1608Metric_Pad1.08x0.95mm_HandSolder
- removed D_{flyback}13, D_{flyback}14: ESD5Z12, Diode_SMD:D_SOD-523
- removed Flywheels_In1, Flywheels_V_{d}1: TestPoint, TestPoint:TestPoint_Keystone_5010-5014_Multipurpose
- removed J_{PA21,LED}1: Conn_01x02, Connector_PinSocket_2.54mm:PinSocket_1x02_P2.54mm_Vertical
- removed M_{flywheel,2}1: Motor_DC, Connector_AMASS:AMASS_XT30U-M_1x02_P5.0mm_Vertical
- removed Q13, Q14, Q21: NTR4501NT1G, ECE445L:SOT96P237X111-3N
- removed R_{I_lim}4: R, Resistor_SMD:R_0603_1608Metric_Pad0.98x0.95mm_HandSolder
- removed R_{choke}13, R_{choke}14: 680, Resistor_SMD:R_0603_1608Metric_Pad0.98x0.95mm_HandSolder
- removed R_{gate}13, R_{gate}14: 0.25, Resistor_SMD:R_0603_1608Metric_Pad0.98x0.95mm_HandSolder
- removed SW_{bypass}13: NO, ECE445L:SW_PUSH_6mm
- added R_{vref}1: 0.5, Resistor_SMD:R_0805_2012Metric_Pad1.20x1.40mm_HandSolder, F.Cu at (137.0, 179.4)
- added R_{vref}2: 0.5, Resistor_SMD:R_0805_2012Metric_Pad1.20x1.40mm_HandSolder, F.Cu at (137.0, 181.7)
- added R_{vref}3: 0.5, Resistor_SMD:R_0805_2012Metric_Pad1.20x1.40mm_HandSolder, B.Cu at (137.0, 179.4)
- added R_{vref}4: 0.5, Resistor_SMD:R_0805_2012Metric_Pad1.20x1.40mm_HandSolder, B.Cu at (137.0, 181.7)
- added U1: DRV8231ADSG, Package_SO:TI_SO-PowerPAD-8, F.Cu at (129.6, 181.2)
- 12V1, 3V3, C_{b}14, J_{IDReader}1, J_{atomizer}1, J_{atomizer}2, Motor_In1, Motor_In11, Motor_In6, Motor_V_{d}1, Motor_V_{d}11, Motor_V_{d}6, RxD_{ID}1, SPI_{CS}1, SPI_{SCK}1, Solenoid_In1, Solenoid_V_{d}1, TxD_{ID}1, uC_{1}←uC_{2}1, uC_{1}→uC_{2}1: moved to B.Cu
- J_{test}1: footprint Connector_PinSocket_2.54mm:PinSocket_2x04_P2.54mm_Vertical -> Connector_PinSocket_2.54mm:PinSocket_1x04_P2.54mm_Vertical
- moved J_{atomizer}1 134.6 mm to (19.8, 59.9), turned to 180 degrees
- moved J_{atomizer}2 134.5 mm to (19.8, 51.2), turned to 180 degrees
- moved J_{test}1 109.7 mm to (138.4, 22.6), turned to 180 degrees
- moved J_{flash}2 107.0 mm to (19.8, 39.9), turned to 180 degrees
- moved Q18 94.5 mm to (131.7, 19.5), turned to 90 degrees
- moved R_{I_lim}1 91.4 mm to (132.0, 15.7), turned to 90 degrees
- moved Q19 90.3 mm to (126.0, 19.3), turned to 90 degrees
- moved J_{PA3,LED}1 88.8 mm to (130.2, 15.1), turned to 180 degrees
- moved R_{I_lim}2 88.0 mm to (126.5, 15.5), turned to 90 degrees
- moved Q20 86.5 mm to (119.2, 19.2), turned to 90 degrees
- moved J_{PA7,LED}1 85.0 mm to (124.5, 14.7), turned to 180 degrees
- moved R_{I_lim}3 84.8 mm to (119.6, 15.5), turned to 90 degrees
- moved C_{b}16 82.7 mm to (58.8, 23.8)
- moved ESP8266 82.7 mm to (55.4, 26.1)
- moved C_{b}17 82.7 mm to (58.9, 23.8)
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- renumbered M_{flywheel,1}1 to M_{winch}1
Connections:
- J_{test}1 pad 2: GND -> PA7/LG2
- J_{test}1 pad 3: PA7/LG2 -> PA14/LG3
- M_{winch}1 pad 1: +12V -> Net-(M_{winch}1-+)
- M_{winch}1 pad 2: /Lab7 Electromech/V_{d,flywheels} -> Net-(M_{winch}1--)
- uC2 pad 28: PA21/LG4 -> Winch_{2}
- uC2 pad 29: Flywheels -> Winch_{1}
Routing:
- net +3V3: track 225.6 -> 982.7 mm, vias 9 -> 11
- net ID Scan - TxD: track 0.00 -> 190.0 mm, vias 0 -> 4
- net ID Scan - RxD: track 0.00 -> 184.7 mm, vias 0 -> 4
- net Solenoid: track 24.0 -> 162.6 mm, vias 0 -> 4
- net Winch_{2}: track 0.00 -> 138.2 mm, vias 0 -> 2
- net Winch_{1}: track 0.00 -> 136.9 mm, vias 0 -> 2
- net /Lab7 Microcontroller/uC_{1} - SWCLK: track 0.00 -> 132.7 mm, vias 0 -> 3
- net /Lab7 Microcontroller/uC_{1} - SWDIO: track 0.00 -> 130.5 mm, vias 0 -> 3
- net Motor PWM: track 0.00 -> 129.8 mm, vias 0 -> 5
- net /Lab7 Microcontroller/uC_{2} - SWDIO: track 0.00 -> 123.0 mm, vias 0 -> 3
- net /Lab7 Microcontroller/uC_{2} - SWCLK: track 0.00 -> 118.4 mm, vias 0 -> 3
- net uC_{1} - ESP RxD: track 0.00 -> 117.2 mm, vias 0 -> 2
- net uC_{1} - ESP Light: track 0.00 -> 117.0 mm, vias 0 -> 2
- net uC_{2} - Speaker: track 0.00 -> 110.3 mm, vias 0 -> 6
- net uC_{1} - ESP TxD: track 0.00 -> 109.7 mm, vias 0 -> 2
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- added copper zone on F.Cu, net /Lab7 Electromech/V_{d,motor 10}
- added copper zone on F.Cu, net /Lab7 Electromech/V_{d,motor 11}
- added copper zone on F.Cu, net /Lab7 Electromech/V_{d,motor 12}
- added copper zone on F.Cu, net /Lab7 Electromech/V_{d,motor 1}
- added copper zone on F.Cu, net /Lab7 Electromech/V_{d,motor 2}
- added copper zone on F.Cu, net /Lab7 Electromech/V_{d,motor 3}
- added copper zone on F.Cu, net /Lab7 Electromech/V_{d,motor 4}
- added copper zone on F.Cu, net /Lab7 Electromech/V_{d,motor 5}
- added copper zone on F.Cu, net /Lab7 Electromech/V_{d,motor 6}
- added copper zone on F.Cu, net /Lab7 Electromech/V_{d,motor 7}
- added copper zone on F.Cu, net /Lab7 Electromech/V_{d,motor 8}
- added copper zone on F.Cu, net /Lab7 Electromech/V_{d,motor 9}
- added copper zone on B.Cu, net /Lab7 Electromech/V_{d,solenoid}
- added copper zone on F.Cu, net /Lab7 Electromech/V_{d,solenoid}
- added copper zone on F.Cu, net GND
- added copper zone on F.Cu, net Net-(M_{winch}1-+)
- added copper zone on F.Cu, net Net-(M_{winch}1--)
- added copper zone on F.Cu, net Net-(Q15-G)
- added copper zone on F.Cu, net Net-(U1-IPROPI)
- removed copper zone on F.Cu, net +3V3
Other:
- board size 147.1 x 184.3 mm -> 147.4 x 184.3 mm
