File: hw/ECE445L_Lab7/ECE445L_Lab7.kicad_pcb (KiCad board)
At the start: 2 copper layers, 147.4 x 184.3 mm, 174 parts, among them M1 Motor_DC, M10 Motor_DC, M11 Motor_DC, M12 Motor_DC, M2 Motor_DC, M3 Motor_DC, M4 Motor_DC, M5 Motor_DC, M6 Motor_DC, M7 Motor_DC, M8 Motor_DC, M9 Motor_DC, Q1 NTR4501NT1G, Q10 NTR4501NT1G, Q11 NTR4501NT1G, Q12 NTR4501NT1G, Q15 NTR4501NT1G, Q16 NTR4501NT1G, Q17 NTR4501NT1G, Q18 NTR4501NT1G, Q19 NTR4501NT1G, Q2 NTR4501NT1G, Q20 NTR4501NT1G, Q3 NTR4501NT1G, Q4 NTR4501NT1G, Q5 NTR4501NT1G, Q6 NTR4501NT1G, Q7 NTR4501NT1G, Q8 NTR4501NT1G, Q9 NTR4501NT1G, U1 DRV8231ADSG, Y1 16MHz, Y2 16MHz

Commit message: resolved some DRC issues
Parts:
- moved J_{USB-C}1 17.5 mm to (97.5, 182.1)
- moved F1 15.5 mm to (89.6, 168.8), turned to 0 degrees
- moved R_{filter}1 5.72 mm to (90.5, 184.0), turned to 90 degrees
- turned C_{filter}1 to 0 degrees
Routing:
- net /Lab7 Power/V_{in,fused}: track 28.4 -> 1.71 mm, vias 0 -> 9
- net GND: track 88.4 -> 66.8 mm, vias 1179 -> 1401
- net /Lab7 Power/V_{in}: track 10.3 -> 0.00 mm
- net +3V3: track 982.7 -> 986.8 mm, vias 11 -> 12
- net Net-(C_{filter}1-Pad1): track 5.97 -> 4.05 mm
- net +12V: vias 135 -> 141
- added copper zone on B.Cu, net /Lab7 Power/V_{in,fused}
- added copper zone on F.Cu, net /Lab7 Power/V_{in,fused}
- added copper zone on B.Cu, net /Lab7 Power/V_{in}
- added copper zone on F.Cu, net /Lab7 Power/V_{in}

Commit message: fixed all drc errors
Parts:
- moved TFT1 1.01 mm to (90.8, 164.8)
- moved J_{IDReader}1 1.00 mm to (161.2, 53.0)
- moved J_{flash}1 1.00 mm to (161.2, 64.5)
- moved TFT2 0.61 mm to (91.3, 40.0)
- moved JP_{Motor}4 0.17 mm to (124.7, 75.1)
- moved JP_{Motor}3 0.15 mm to (124.7, 92.4)
- moved R_{gate}4 0.07 mm to (127.2, 74.9)
- moved JP_{Motor}2 0.06 mm to (56.6, 75.7)
Routing:
- net Motor_{8}: track 38.3 -> 36.2 mm
- net Motor_{11}: track 75.2 -> 73.4 mm
- net Motor_{9}: track 49.4 -> 47.7 mm
- net /Lab7 IO/D_{Motor}3: track 92.2 -> 90.5 mm
- net /Lab7 IO/D_{Motor}4: track 100.4 -> 98.7 mm
- net HLG Screen - MOSI: track 37.2 -> 38.7 mm
- net HiLetGo - SCK: track 27.9 -> 29.1 mm
- net Adafruit - CS: track 29.9 -> 30.9 mm
- net ID Scan - TxD: track 190.0 -> 189.0 mm
- net ID Scan - RxD: track 184.7 -> 183.7 mm
- net /Lab7 Microcontroller/uC_{1} - SWDIO: track 130.5 -> 129.5 mm
- net /Lab7 Microcontroller/uC_{1} - SWCLK: track 133.0 -> 132.0 mm
- net Adafruit - RST: track 38.5 -> 39.4 mm
- net HLG SDC - MISO: track 25.7 -> 26.4 mm
- net Adafruit - D/C: track 43.5 -> 44.2 mm
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