File: hw/ECE445L_Lab7/ECE445L_Lab7.kicad_pcb (KiCad board)
At the start: 2 copper layers, 147.4 x 184.3 mm, 174 parts, among them M1 Motor_DC, M10 Motor_DC, M11 Motor_DC, M12 Motor_DC, M2 Motor_DC, M3 Motor_DC, M4 Motor_DC, M5 Motor_DC, M6 Motor_DC, M7 Motor_DC, M8 Motor_DC, M9 Motor_DC, Q1 NTR4501NT1G, Q10 NTR4501NT1G, Q11 NTR4501NT1G, Q12 NTR4501NT1G, Q15 NTR4501NT1G, Q16 NTR4501NT1G, Q17 NTR4501NT1G, Q18 NTR4501NT1G, Q19 NTR4501NT1G, Q2 NTR4501NT1G, Q20 NTR4501NT1G, Q3 NTR4501NT1G, Q4 NTR4501NT1G, Q5 NTR4501NT1G, Q6 NTR4501NT1G, Q7 NTR4501NT1G, Q8 NTR4501NT1G, Q9 NTR4501NT1G, U1 DRV8231ADSG, Y1 16MHz, Y2 16MHz

Commit message: minor tweaks
Routing:
- net +3V3: track 986.7 -> 984.8 mm
- net GND: vias 1474 -> 1519
