File: hw/ECE445L_Lab7/Lab7_Input.kicad_sch (KiCad schematic)
At the start: 32 parts, among them Q16 NTR4501NT1G, Q17 NTR4501NT1G, Q18 NTR4501NT1G, Q19 NTR4501NT1G, Q20 NTR4501NT1G, Q21 NTR4501NT1G

Commit message: finished prelim layout for TA review
Parts:
- removed J_{PA21,LED}1: Conn_01x02, Connector_PinSocket_2.54mm:PinSocket_1x02_P2.54mm_Vertical, symbol Connector_Generic:Conn_01x02
- removed Q21: NTR4501NT1G, ECE445L:SOT96P237X111-3N, symbol ECE445L:NTR4501NT1G
- removed R_{I_lim}4: R, Resistor_SMD:R_0603_1608Metric_Pad0.98x0.95mm_HandSolder, symbol Device:R
